File: Production/Qwiic Board/SparkFun_tDof-TMF8820-Panel.brd (EAGLE design)
At the start: 175 x 117.3 mm, 1350 parts, among them J10 QWIIC_RIGHT_ANGLE, J13 QWIIC_RIGHT_ANGLE, J14 QWIIC_RIGHT_ANGLE, J17 QWIIC_RIGHT_ANGLE, J18 QWIIC_RIGHT_ANGLE, J2 QWIIC_RIGHT_ANGLE, J21 QWIIC_RIGHT_ANGLE, J22 QWIIC_RIGHT_ANGLE, J25 QWIIC_RIGHT_ANGLE, J26 QWIIC_RIGHT_ANGLE, J29 QWIIC_RIGHT_ANGLE, J3 QWIIC_RIGHT_ANGLE, J30 QWIIC_RIGHT_ANGLE, J33 QWIIC_RIGHT_ANGLE, J34 QWIIC_RIGHT_ANGLE, J37 QWIIC_RIGHT_ANGLE, J38 QWIIC_RIGHT_ANGLE, J4 QWIIC_RIGHT_ANGLE, J41 QWIIC_RIGHT_ANGLE, J42 QWIIC_RIGHT_ANGLE, J45 QWIIC_RIGHT_ANGLE, J46 QWIIC_RIGHT_ANGLE, J49 QWIIC_RIGHT_ANGLE, J5 QWIIC_RIGHT_ANGLE, J50 QWIIC_RIGHT_ANGLE, J53 QWIIC_RIGHT_ANGLE, J54 QWIIC_RIGHT_ANGLE, J57 QWIIC_RIGHT_ANGLE, J58 QWIIC_RIGHT_ANGLE, J61 QWIIC_RIGHT_ANGLE, J62 QWIIC_RIGHT_ANGLE, J65 QWIIC_RIGHT_ANGLE, J66 QWIIC_RIGHT_ANGLE, J69 QWIIC_RIGHT_ANGLE, J70 QWIIC_RIGHT_ANGLE, J73 QWIIC_RIGHT_ANGLE, J74 QWIIC_RIGHT_ANGLE, J77 QWIIC_RIGHT_ANGLE, J78 QWIIC_RIGHT_ANGLE, J81 QWIIC_RIGHT_ANGLE, J82 QWIIC_RIGHT_ANGLE, J85 QWIIC_RIGHT_ANGLE, J86 QWIIC_RIGHT_ANGLE, J89 QWIIC_RIGHT_ANGLE, J9 QWIIC_RIGHT_ANGLE, J90 QWIIC_RIGHT_ANGLE, J93 QWIIC_RIGHT_ANGLE, J94 QWIIC_RIGHT_ANGLE

Commit message: Adds new panel with corrected silk
Parts:
- U$120, U$150, U$180, U$19, U$210, U$240, U$270, U$300, U$330, U$360, U$390, U$420, U$450, U$480, U$510, U$540, U$570, U$60, U$600, U$630, U$660, U$690, U$720, U$90: device TMFBot:#GP0#8 -> TMFBot:#GP1#8
- moved U$630 2.54 mm to (73.4, 81.4)
- moved U$270 2.54 mm to (73.4, 29.6)
- moved U$90 2.54 mm to (73.4, 3.68)
- moved U$450 2.54 mm to (73.4, 55.5)
- moved U$570 2.54 mm to (21.6, 81.4)
- moved U$600 2.54 mm to (47.5, 81.4)
- moved U$19 2.54 mm to (21.6, 3.68)
- moved U$210 2.54 mm to (21.6, 29.6)
- moved U$240 2.54 mm to (47.5, 29.6)
- moved U$60 2.54 mm to (47.5, 3.68)
- moved U$390 2.54 mm to (21.6, 55.5)
- moved U$420 2.54 mm to (47.5, 55.5)
- moved U$660 2.54 mm to (99.3, 81.4)
- moved U$690 2.54 mm to (125.2, 81.4)
- moved U$720 2.54 mm to (151.1, 81.4)
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